File: SpinPixel.kicad_sch (KiCad schematic)
At the start: 1 part

Commit message: capacitor
Parts:
- added C1: C, symbol Device:C
Changed lines of the file:
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@@
 (kicad_sch (version 20230121) (generator eeschema)
   (paper "A4")
+  (symbol (lib_id "Device:C") (at 118.11 76.2 0) (unit 1)
+    (in_bom yes) (on_board yes) (dnp no) (fields_autoplaced)
+    (property "Reference" "C1" (at 121.92 74.93 0)
+      (effects (font (size 1.27 1.27)) (justify left))
+    )
+    (property "Value" "C" (at 121.92 77.47 0)
+      (effects (font (size 1.27 1.27)) (justify left))
+    )
+    (property "Footprint" "" (at 119.0752 80.01 0)
+      (effects (font (size 1.27 1.27)) hide)
+    )
+    (property "Datasheet" "~" (at 118.11 76.2 0)
+      (effects (font (size 1.27 1.27)) hide)
+    )
+    (pin "1")
+    (pin "2")
+    (instances
+      (project "SpinPixel"
+        (path "/00b468ec-61f9-4c5d-bec4-a351a57d98e5"
+          (reference "C1") (unit 1)
+        )
+      )
+    )
+  )
   (symbol (lib_id "Device:R") (at 147.32 97.79 0) (unit 1)
     (in_bom yes) (on_board yes) (dnp no) (fields_autoplaced)

Commit message: Test2
Parts:
- added L1: L, symbol Device:L
Changed lines of the file:
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@@
+    )
+  )
+  (symbol (lib_id "Device:L") (at 133.35 95.25 0) (unit 1)
+    (in_bom yes) (on_board yes) (dnp no) (fields_autoplaced)
+    (property "Reference" "L1" (at 134.62 94.615 0)
+      (effects (font (size 1.27 1.27)) (justify left))
+    )
+    (property "Value" "L" (at 134.62 97.155 0)
+      (effects (font (size 1.27 1.27)) (justify left))
+    )
+    (property "Footprint" "" (at 133.35 95.25 0)
+      (effects (font (size 1.27 1.27)) hide)
+    )
+    (property "Datasheet" "~" (at 133.35 95.25 0)
+      (effects (font (size 1.27 1.27)) hide)
+    )
+    (pin "1")
+    (pin "2")
+    (instances
+      (project "SpinPixel"
+        (path "/00b468ec-61f9-4c5d-bec4-a351a57d98e5"
+          (reference "L1") (unit 1)
+        )
+      )
     )
   )

Commit message: c2
Parts:
- added C2: C, symbol Device:C
Changed lines of the file:
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@@
+    )
+  )
+  (symbol (lib_id "Device:C") (at 118.11 88.9 0) (unit 1)
+    (in_bom yes) (on_board yes) (dnp no) (fields_autoplaced)
+    (property "Reference" "C2" (at 121.92 87.63 0)
+      (effects (font (size 1.27 1.27)) (justify left))
+    )
+    (property "Value" "C" (at 121.92 90.17 0)
+      (effects (font (size 1.27 1.27)) (justify left))
+    )
+    (property "Footprint" "" (at 119.0752 92.71 0)
+      (effects (font (size 1.27 1.27)) hide)
+    )
+    (property "Datasheet" "~" (at 118.11 88.9 0)
+      (effects (font (size 1.27 1.27)) hide)
+    )
+    (pin "1")
+    (pin "2")
+    (instances
+      (project "SpinPixel"
+        (path "/00b468ec-61f9-4c5d-bec4-a351a57d98e5"
+          (reference "C2") (unit 1)
+        )
+      )
     )
   )
